File: nol.board-feather.brd (EAGLE design)
At the start: 63.5 x 22.9 mm, 34 parts, among them J11 ZX62-B-5PA, J5 4P-SMD-2.0-90D, J6 GREEN-2P-3.5 (NC), SW1 SPST_TACT-KMR2, SW2 SPST_TACT-KMR2, U1 FT230XS-R-SSOP16, U2 AP2112K-3.3, U3 MCP73831T-2ACI/OT, U4 PLM-12X2

Commit message: DK-1 Added BOM. Finished with order.
Parts:
- added U$1: COXLAB5X5MM, coxlab:COXLAB_5X5MM
- added U$7: NOLA10X10MM, coxlab:NOLA_10X10MM
Other:
- board text added: "!CHG"
- board text added: "!RESET"
- board text added: "+3V"
- board text added: "1"
- board text added: "10"
- board text added: "11"
- board text added: "13"
- board text added: "14"
- board text added: "15"
- board text added: "16"
- board text added: "17"
- board text added: "18"
- board text added: "2"
- board text added: "3"
- board text added: "4"
- board text added: "5"
- board text added: "6"
- board text added: "7"
- board text added: "8"
- board text added: "9"
- board text added: "EN"
- board text added: "GND"
- board text added: "J_TEST"
- board text added: "NC"
- board text added: "Nol.Board-Feather Rev. 0"
- board text added: "REF"
- board text added: "VBAT"
- board text added: "VBUS"
- board text added: "by"
- board text removed: "Nol.Board-Feather by CoXlab Inc."
