File: nol.board-feather.sch (EAGLE design)
At the start: 34 parts, among them J11 ZX62-B-5PA, J5 4P-SMD-2.0-90D, J6 GREEN-2P-3.5 (NC), SW1 SPST_TACT-KMR2, SW2 SPST_TACT-KMR2, U1 FT230XS-R-SSOP16, U2 AP2112K-3.3, U3 MCP73831T-2ACI/OT, U4 PLM-12X2

Commit message: DK-1 Added BOM. Finished with order.
Parts:
- added U$1: COXLAB5X5MM, coxlab:COXLAB5X5MM
- added U$7: NOLA10X10MM, coxlab:NOLA10X10MM
Changed lines of the file:
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@@
 <setting verticaltext="up"/>
 </settings>
-<grid distance="0.1" unitdist="inch" unit="inch" style="lines" multiple="1" display="no" altdistance="0.05" altunitdist="inch" altunit="inch"/>
+<grid distance="0.1" unitdist="inch" unit="inch" style="lines" multiple="1" display="no" altdistance="0.01" altunitdist="inch" altunit="inch"/>
 <layers>
 <layer number="1" name="Top" color="4" fill="1" visible="no" active="no"/>
@@
 <part name="+3V1" library="supply1" deviceset="+3V3" device=""/>
 <part name="GND7" library="supply1" deviceset="GND" device=""/>
-<part name="SW1" library="adafruit" deviceset="SPST_TACT" device="-KMR2"/>
+<part name="SW1" library="adafruit" library_urn="urn:adsk.eagle:library:420" deviceset="SPST_TACT" device="-KMR2" package3d_urn="urn:adsk.eagle:package:6240885/1"/>
 <part name="GND3" library="supply1" library_urn="urn:adsk.eagle:library:371" deviceset="GND" device=""/>
 <part name="GND4" library="supply1" library_urn="urn:adsk.eagle:library:371" deviceset="GND" device=""/>
@@
 <part name="GND6" library="supply1" library_urn="urn:adsk.eagle:library:371" deviceset="GND" device=""/>
 <part name="GND8" library="supply1" deviceset="GND" device=""/>
-<part name="SW2" library="adafruit" deviceset="SPST_TACT" device="-KMR2"/>
+<part name="SW2" library="adafruit" library_urn="urn:adsk.eagle:library:420" deviceset="SPST_TACT" device="-KMR2" package3d_urn="urn:adsk.eagle:package:6240885/1"/>
 <part name="C2" library="microbuilder" deviceset="CAP_CERAMIC" device="0805-NOOUTLINE" value="10µF"/>
 <part name="C4" library="microbuilder" deviceset="CAP_CERAMIC" device="0805-NOOUTLINE" value="100nF"/>
@@
 <part name="GND14" library="supply1" library_urn="urn:adsk.eagle:library:371" deviceset="GND" device=""/>
 <part name="+3V5" library="supply1" deviceset="+3V3" device=""/>
+<part name="U$1" library="coxlab" deviceset="COXLAB" device="5X5MM" value="COXLAB5X5MM"/>
+<part name="U$7" library="coxlab" deviceset="NOLA" device="10X10MM"/>
 </parts>
 <sheets>
@@
 <attribute name="VALUE" x="118.11" y="137.16" size="1.778" layer="96" rot="MR0"/>
 </instance>
+<instance part="U$1" gate="G$1" x="261.62" y="10.16" smashed="yes"/>
+<instance part="U$7" gate="G$1" x="261.62" y="15.24" smashed="yes"/>
 </instances>
 <busses>
